Commit message: Roboboat base_link floats in Gazebo. Need to add sensors, actuators.

File: roboboat/roboboat_description/urdf/actuators.xacro (robot description, xacro)
@@ -8,20 +8,11 @@
           aware that Gazebo does not use the SNAME convention per default.
     -->
-    <!-- TODO: Adjust these based on Gazebo Visual with CAD model -->
-    <!-- Port Bow Thruster -->
+    <!-- Right Thruster -->
     <xacro:thruster_macro robot_namespace="$(arg namespace)" suffix_ns="$(arg suffix_ns)" thruster_id="0">
-        <origin xyz="-0.53 -0.377654 -0.16" rpy="0 0 0.785398163" />
+        <origin xyz="-0.53 -0.377654 -0.16" rpy="0 0 0" />
     </xacro:thruster_macro>
-    <!-- Starboard Bow Thruster -->
+    <!-- Left Thruster -->
     <xacro:thruster_macro robot_namespace="$(arg namespace)" suffix_ns="$(arg suffix_ns)" thruster_id="1">
-        <origin xyz="-0.53 0.377654 -0.16" rpy="0 0 -0.785398163" />
-    </xacro:thruster_macro>
-    <!-- Port Stern Thruster -->
-    <xacro:thruster_macro robot_namespace="$(arg namespace)" suffix_ns="$(arg suffix_ns)" thruster_id="2">
-        <origin xyz="-0.53 -0.377654 -0.16" rpy="0 0 0.785398163" />
-    </xacro:thruster_macro>
-    <!-- Starboard Stern Thruster -->
-    <xacro:thruster_macro robot_namespace="$(arg namespace)" suffix_ns="$(arg suffix_ns)" thruster_id="3">
-        <origin xyz="-0.53 0.377654 -0.16" rpy="0 0 -0.785398163" />
+        <origin xyz="-0.53 0.377654 -0.16" rpy="0 0 0" />
     </xacro:thruster_macro>
 </robot>

File: roboboat/roboboat_description/urdf/base.xacro (robot description, xacro)
@@ -1,70 +1,71 @@
 <?xml version="1.0"?>
 <robot xmlns:xacro="http://www.ros.org/wiki/xacro">
-	<xacro:property name="mass" value="22.69"/> <!-- TODO: Adjust this to actual vessel mass: approximately 50/2.204 kg -->
-	<!-- Center of gravity -->
-	<xacro:property name="cog" value="0 0 0"/> <!-- TODO: Adjust this to be NEGATIVE DRAFT from roboboat_gazebo/launch/roboboat_sim.launch -->
-	<!-- Fluid density -->
-	<xacro:property name="rho" value="1000"/>
-	<!-- Loading vehicle's specific macros -->
-	<xacro:include filename="$(find roboboat_description)/urdf/snippets.xacro"/>
-	<!-- Define a color -->
-	<material name="dark_gray"><color rgba="0.2 0.2 0.2 1.0"/></material>
-	<!-- Vehicle macro -->
-  	<xacro:macro name="roboboat_base" params="namespace *gazebo">
-		<!-- Rigid body description of the base link -->
-		<link name="${namespace}base_link">
-		<!--
-		Be careful to setup the coefficients for the inertial tensor,
-		otherwise your model will become unstable on Gazebo
-		-->
-			<visual>
-	          <origin xyz="0 0 0" rpy="1.570796327 0 0"/>
-	          <geometry>
-	            <mesh filename="package://roboboat_description/meshes/Final-Catamaran.stl" scale="1 1 1" />
-	          </geometry>
-	          <material name="dark_gray" />
-	        </visual>
-	        <collision>
-	          <origin xyz="0 0 0" rpy="0 0 0"/>
-	          <geometry>
-	            <mesh filename="package://roboboat_description/meshes/Final-Catamaran.stl" scale="1 1 1" />
-	          </geometry>
-	        </collision>
-      	</link>
-      	<!-- Dummy Link to contain the inertial information for base_link -->
-		<link name="${namespace}dummy_link">
-			<inertial>
-				  <mass value="${mass}" />
-				  <origin xyz="${cog}" rpy="0 0 0"/>
-				  <inertia ixx="22.59" ixy="0" iyy = "22.59" ixz="0" iyz="0" izz="10" />
-				  <!-- <inertia ixx="0.017474" ixy="-0.000013" ixz="-0.000102"
-				                          iyy="0.017781"  iyz="-0.000058"
-				                                          izz="0.033235" /> -->
-			</inertial>
-		</link>
-		<!-- Join the dummy frame and the base_link frames -->
-		<joint name="dummy_to_base" type="fixed">
-	        <parent link="${namespace}base_link" />
-	        <child link="${namespace}dummy_link" />
-	    </joint>
-		<gazebo reference="${namespace}base_link">
-		  <selfCollide>false</selfCollide>
-		  <material>Gazebo/DarkGrey</material>
-		  <gravity>1</gravity>
-		</gazebo>
-		<!-- Set up hydrodynamic plugin given as input parameter -->
-    	<xacro:insert_block name="gazebo"/>
-	    <!-- Include the thruster modules -->
-	    <xacro:include filename="$(find roboboat_description)/urdf/actuators.xacro"/>
-	    <!-- Include the sensor modules -->
-	    <xacro:include filename="$(find roboboat_description)/urdf/sensors.xacro"/>
-	    <!-- BA  5/18/2020: I don't think we need this
-	    <xacro:include filename="$(find roboboat_description)/urdf/accessories.urdf.xacro" />
-		-->
-		<!-- BA 5/18/2020: Or this -->
-	    <!-- Optional custom includes. -->
-	    <!--
-	    <xacro:include filename="$(optenv ROBOBOAT_URDF_EXTRAS empty.urdf)" />
-	    -->
-	  </xacro:macro>
+  <!--
+    Vehicle's parameters (remember to enter the model parameters below)
+  -->
+  <xacro:property name="mass" value="31.76"/>
+  <!-- Center of gravity -->
+  <xacro:property name="cog" value="0 0 -0.13"/> <!-- TODO: Check this value -->
+  <!-- Fluid density -->
+  <xacro:property name="rho" value="1000"/>
+  <!-- Loading vehicle's specific macros -->
+  <!--
+  <xacro:include filename="$(find roboboat_description)/urdf/snippets.xacro"/>
+  -->
+  <material name="gray"><color rgba="0.7 0.7 0.7 1.0"/></material>
+  <material name="dark_gray"><color rgba="0.2 0.2 0.2 1.0"/></material>
+  <material name="yellow"><color rgba="0.8 0.8 0.0 1.0"/></material>
+  <!-- Vehicle macro -->
+  <xacro:macro name="roboboat_base" params="namespace *gazebo">
+      <!-- Rigid body description of the base link -->
+      <link name="${namespace}base_link">
+        <!--
+          Be careful to setup the coefficients for the inertial tensor,
+          otherwise your model will become unstable on Gazebo
+        -->
+        <visual>
+          <origin xyz="0 0 0" rpy="0 0 0"/>
+          <geometry>
+            <mesh filename="package://roboboat_description/meshes/base_link.STL" scale="1 1 1" />
+          </geometry>
+          <material name="dark_gray" />
+        </visual>
+        <collision>
+          <origin xyz="0 0 0" rpy="0 0 0"/>
+          <geometry>
+            <mesh filename="package://roboboat_description/meshes/base_link.STL" scale="1 1 1" />
+          </geometry>
+        </collision>
+      </link>
+      <!-- Dummy Link to contain the inertial information for base_link -->
+      <link name="${namespace}dummy_link">
+        <inertial>
+          <mass value="${mass}" />
+          <origin xyz="${cog}" rpy="0 0 0"/>
+          <inertia ixx="10" ixy="0" iyy = "10" ixz="0" iyz="0" izz="10" />
+          <!-- <inertia ixx="0.017474" ixy="-0.000013" ixz="-0.000102"
+                                  iyy="0.017781"  iyz="-0.000058"
+                                                  izz="0.033235" /> -->
+        </inertial>
+      </link>
+      <joint name="dummy_to_base" type="fixed">
+        <parent link="${namespace}base_link" />
+        <child link="${namespace}dummy_link" />
+      </joint>
+    <gazebo reference="${namespace}base_link">
+      <selfCollide>false</selfCollide>
+      <material>Gazebo/DarkGrey</material>
+      <gravity>1</gravity>
+    </gazebo>
+    <!-- Set up hydrodynamic plugin given as input parameter -->
+    <xacro:insert_block name="gazebo"/>
+    <!-- Include the thruster modules -->
+    <!--
+    <xacro:include filename="$(find roboboat_description)/urdf/actuators.xacro"/>
+    -->
+    <!-- Include the sensor modules -->
+    <xacro:include filename="$(find roboboat_description)/urdf/sensors.xacro"/>
+    <!-- Optional custom includes. -->
+    <xacro:include filename="$(optenv roboboat_URDF_EXTRAS empty.urdf)" />
+  </xacro:macro>
 </robot>

File: roboboat/roboboat_description/urdf/gazebo.xacro (robot description, xacro)
@@ -4,10 +4,9 @@
     <xacro:property name="roboboat_cob" value="0 0 0"/>
     <!-- Vehicle's actual volume (Gazebo cannot compute the volume out of the mesh) -->
-    <!-- TODO: This is an estimate -->
-    <xacro:property name="roboboat_volume" value="0.27"/>
+    <xacro:property name="roboboat_volume" value="0.13"/>
     <!-- Describing the dimensions of the vehicle's bounding box -->
-    <xacro:property name="roboboat_length" value="1.524"/>
-    <xacro:property name="roboboat_width"  value="0.8123"/>
-    <xacro:property name="roboboat_height" value="0.254"/>
+    <xacro:property name="roboboat_length" value="1.35"/>
+    <xacro:property name="roboboat_width"  value="1.0"/>
+    <xacro:property name="roboboat_height" value="0.32"/>
     <xacro:macro name="roboboat_hydro_model" params="namespace">
       <!-- List of hydrodynamic models this robot's links -->
@@ -24,8 +23,7 @@
                    buoyancy force computation for the surface vessel.
               -->
-              <!-- TODO: What do these represent? -->
               <metacentric_width>0.1</metacentric_width>
               <metacentric_length>0.1</metacentric_length>
-              <submerged_height>0.0635</submerged_height> <!-- TODO: Get this more accurate -->
+              <submerged_height>0.02</submerged_height>
               <hydrodynamic_model>
                   <type>fossen</type>
@@ -39,5 +37,4 @@
                 </added_mass>
                 <offset_added_mass>0</offset_added_mass>
-                  <!-- TODO: This is default from Heron. Update -->
                   <linear_damping>
                       -16.44998712 -15.79776044 -100 -13 -13 -6

File: roboboat/roboboat_description/urdf/sensors.xacro (robot description, xacro)
@@ -18,5 +18,4 @@
   </gazebo>
   <link name="$(arg suffix_ns)navsat_link" />
-  <!-- TODO: Find these environment variables: ROBOBOAT_NAVSAT_UBLOX_XYZ, ROBOBOAT_NAVSAT_UBLOX_RPY -->
   <joint name="navsat_joint" type="fixed">
     <parent link="$(arg suffix_ns)base_link" />
@@ -24,23 +23,22 @@
     <origin xyz="$(optenv ROBOBOAT_NAVSAT_UBLOX_XYZ 0.015 0.050 0.072)"
       rpy="$(optenv ROBOBOAT_NAVSAT_UBLOX_RPY 0.0 0.0 0.0)" />
-  </joint>
-  <!-- IMU -->
-  <gazebo>
-    <plugin name="imu_controller" filename="libhector_gazebo_ros_imu.so">
-      <robotNamespace>/$(arg namespace)</robotNamespace>
-      <updateRate>50.0</updateRate>
-      <bodyName>$(arg suffix_ns)imu_link</bodyName>
-      <frameId>$(arg suffix_ns)imu_link</frameId>
-      <topicName>/$(arg suffix_ns)imu/data_raw</topicName>
-      <accelDrift>0.005 0.005 0.005</accelDrift>
-      <accelGaussianNoise>0.005 0.005 0.005</accelGaussianNoise>
-      <rateDrift>0.005 0.005 0.005 </rateDrift>
-      <rateGaussianNoise>0.005 0.005 0.005 </rateGaussianNoise>
-      <headingDrift>0.005</headingDrift>
-      <headingGaussianNoise>0.005</headingGaussianNoise>
-    </plugin>
-  </gazebo>
+    </joint>
+    <!-- IMU -->
+    <gazebo>
+      <plugin name="imu_controller" filename="libhector_gazebo_ros_imu.so">
+        <robotNamespace>/$(arg namespace)</robotNamespace>
+        <updateRate>50.0</updateRate>
+        <bodyName>$(arg suffix_ns)imu_link</bodyName>
+        <frameId>$(arg suffix_ns)imu_link</frameId>
+        <topicName>/$(arg suffix_ns)imu/data_raw</topicName>
+        <accelDrift>0.005 0.005 0.005</accelDrift>
+        <accelGaussianNoise>0.005 0.005 0.005</accelGaussianNoise>
+        <rateDrift>0.005 0.005 0.005 </rateDrift>
+        <rateGaussianNoise>0.005 0.005 0.005 </rateGaussianNoise>
+        <headingDrift>0.005</headingDrift>
+        <headingGaussianNoise>0.005</headingGaussianNoise>
+      </plugin>
+    </gazebo>
     <link name="$(arg suffix_ns)imu_link" />
-    <!-- TODO: Find these environment variables: ROBOBOAT_IMU_UM6_XYZ, ROBOBOAT_IMU_UM6_RPY -->
     <joint name="$(arg suffix_ns)imu_joint" type="fixed">
       <origin xyz="$(optenv ROBOBOAT_IMU_UM6_XYZ -0.1397 0.0 0)" rpy="$(optenv ROBOBOAT_IMU_UM6_RPY 0 0.0 0.0)" />
@@ -48,4 +46,17 @@
       <child link="$(arg suffix_ns)imu_link" />
     </joint>
+    <!-- Magnetometer -->
+    <gazebo>
+      <plugin name="mag_controller" filename="libhector_gazebo_ros_magnetic.so">
+        <updateRate>50</updateRate>
+        <robotNamespace>/$(arg namespace)</robotNamespace>
+        <bodyName>$(arg suffix_ns)imu_link</bodyName>
+        <frameId>$(arg suffix_ns)imu_link</frameId>
+        <topicName>/$(arg suffix_ns)imu/mag</topicName>
+        <referenceHeading>90</referenceHeading>
+        <drift>0.0005 0.0005 0.0005</drift>
+        <gaussianNoise>0.025 0.025 0.025</gaussianNoise>
+      </plugin>
+    </gazebo>
     <!-- Mount a Perfect Pose 3D sensor. -->
     <gazebo>
@@ -59,4 +70,3 @@
       </plugin>
     </gazebo>
-  <!-- Mount a ZED (or 2) -->
-</robot>
+  </robot>

File: roboboat/roboboat_description/urdf/snippets.xacro (robot description, xacro)
@@ -1,5 +1,5 @@
 <?xml version="1.0"?>
 <robot xmlns:xacro="http://www.ros.org/wiki/xacro">
-	<!-- MACRO FOR THRUSTER UNITS  -->
+  <!-- MACRO FOR THRUSTER UNITS  -->
   <!--
     Thruster macro with integration of joint and link. The thrusters should
@@ -15,5 +15,5 @@
       <visual>
         <geometry>
-          <mesh filename="package://roboboat_description/meshes/Rugged-Thruster (Modified).stl" scale="1 1 1" />
+          <mesh filename="package://roboboat_description/meshes/prop.dae" scale="1 1 1" />
         </geometry>
       </visual>
@@ -49,8 +49,6 @@
         <clampMin>-100</clampMin>
         <!-- Minimum and maximum thrust force output allowed -->
-        <!-- Found from scaling the KgF values to Newtons from: https://bluerobotics.com/store/thrusters/t100-t200-thrusters/t200-thruster/ -->
-        <!-- Using 16V performance curve -->
-        <thrustMin>-40</thrustMin>
-        <thrustMax>51.5</thrustMax>
+        <thrustMin>-35</thrustMin>
+        <thrustMax>35</thrustMax>
         <!--
         Value from 0 to 1 to set the efficiency of the output thrust force
@@ -79,5 +77,5 @@
           <type>LinearInterp</type>
           <inputValues>-1.0 -0.8 -0.6 -0.4 -0.2 0 0.2 0.4 0.6 0.8 1.0</inputValues>
-          <outputValues>-39.1 -29.32 -19.02 -10.00 -3.14 0.0 3.92 12.55 23.83 37.46 51.5</outputValues>
+          <outputValues>-19.88 -16.52 -12.6 -5.6 -1.4 0.0 2.24 9.52 21.28 28.0 33.6</outputValues>
         </conversion>
       </plugin>

Commit message: Spawning actuators in correct orientation. Do not appear to move with hull.

File: roboboat/roboboat_description/urdf/actuators.xacro (robot description, xacro)
@@ -8,11 +8,19 @@
           aware that Gazebo does not use the SNAME convention per default.
     -->
-    <!-- Right Thruster -->
+    <!-- Port Bow -->
     <xacro:thruster_macro robot_namespace="$(arg namespace)" suffix_ns="$(arg suffix_ns)" thruster_id="0">
-        <origin xyz="-0.53 -0.377654 -0.16" rpy="0 0 0" />
+        <origin xyz="-0.27569 0.32286 -0.29202" rpy="1.570796327 0 2.35619449" />
     </xacro:thruster_macro>
-    <!-- Left Thruster -->
+    <!-- Starboard Bow -->
     <xacro:thruster_macro robot_namespace="$(arg namespace)" suffix_ns="$(arg suffix_ns)" thruster_id="1">
-        <origin xyz="-0.53 0.377654 -0.16" rpy="0 0 0" />
+        <origin xyz="0.27569 0.32286 -0.29202" rpy="1.570796327 0 -2.35619449" />
+    </xacro:thruster_macro>
+    <!-- Port Stern -->
+    <xacro:thruster_macro robot_namespace="$(arg namespace)" suffix_ns="$(arg suffix_ns)" thruster_id="2">
+        <origin xyz="-0.28311 -0.31544 -0.29202" rpy="1.570796327 0 -2.35619449" />
+    </xacro:thruster_macro>
+    <!-- Starboard Stern -->
+    <xacro:thruster_macro robot_namespace="$(arg namespace)" suffix_ns="$(arg suffix_ns)" thruster_id="3">
+        <origin xyz="0.28311 -0.31544 -0.29202" rpy="1.570796327 0 2.35619449" />
     </xacro:thruster_macro>
 </robot>

File: roboboat/roboboat_description/urdf/base.xacro (robot description, xacro)
@@ -10,7 +10,5 @@
   <xacro:property name="rho" value="1000"/>
   <!-- Loading vehicle's specific macros -->
-  <!--
   <xacro:include filename="$(find roboboat_description)/urdf/snippets.xacro"/>
-  -->
   <material name="gray"><color rgba="0.7 0.7 0.7 1.0"/></material>
   <material name="dark_gray"><color rgba="0.2 0.2 0.2 1.0"/></material>
@@ -44,7 +42,4 @@
           <origin xyz="${cog}" rpy="0 0 0"/>
           <inertia ixx="10" ixy="0" iyy = "10" ixz="0" iyz="0" izz="10" />
-          <!-- <inertia ixx="0.017474" ixy="-0.000013" ixz="-0.000102"
-                                  iyy="0.017781"  iyz="-0.000058"
-                                                  izz="0.033235" /> -->
         </inertial>
       </link>
@@ -61,7 +56,5 @@
     <xacro:insert_block name="gazebo"/>
     <!-- Include the thruster modules -->
-    <!--
     <xacro:include filename="$(find roboboat_description)/urdf/actuators.xacro"/>
-    -->
     <!-- Include the sensor modules -->
     <xacro:include filename="$(find roboboat_description)/urdf/sensors.xacro"/>

File: roboboat/roboboat_description/urdf/snippets.xacro (robot description, xacro)
@@ -15,13 +15,27 @@
       <visual>
         <geometry>
-          <mesh filename="package://roboboat_description/meshes/prop.dae" scale="1 1 1" />
+          <mesh filename="package://roboboat_description/meshes/base_link_to_port_bow.STL" />
         </geometry>
+        <material
+          name="">
+          <color
+            rgba="0.79216 0.81961 0.93333 1" />
+        </material>
       </visual>
+      <!--Is this causing some rotation? -->
+      <!-- Actuators not moving with hull -->
       <inertial>
-        <mass value="0.001" />
-        <origin xyz="0 0 0" rpy="0 0 0"/>
-        <inertia ixx="0.000000017" ixy="0.0" ixz="0.0"
-               iyy="0.000000017" iyz="0.0"
-               izz="0.000000017" />
+        <origin
+          xyz="0 0 0"
+          rpy="0 0 0" />
+        <mass
+          value="0.19483" />
+        <inertia
+          ixx="0.00013116"
+          ixy="8.7805E-08"
+          ixz="-1.5186E-07"
+          iyy="0.00012713"
+          iyz="-1.4655E-07"
+          izz="0.00018124" />
       </inertial>
     </link>
@@ -29,5 +43,5 @@
     <joint name="${suffix_ns}thruster_${thruster_id}_joint" type="continuous">
       <xacro:insert_block name="origin" />
-      <axis xyz="1 0 0" />
+      <axis xyz="0 0 1" />
       <parent link="${suffix_ns}base_link" />
       <child link="${suffix_ns}thruster_${thruster_id}" />
@@ -49,6 +63,8 @@
         <clampMin>-100</clampMin>
         <!-- Minimum and maximum thrust force output allowed -->
-        <thrustMin>-35</thrustMin>
-        <thrustMax>35</thrustMax>
+        <!-- Found from scaling the KgF values to Newtons from: https://bluerobotics.com/store/thrusters/t100-t200-thrusters/t200-thruster/ -->
+        <!-- Using 16V performance curve -->
+        <thrustMin>-40</thrustMin>
+        <thrustMax>51.5</thrustMax>
         <!--
         Value from 0 to 1 to set the efficiency of the output thrust force
@@ -77,5 +93,5 @@
           <type>LinearInterp</type>
           <inputValues>-1.0 -0.8 -0.6 -0.4 -0.2 0 0.2 0.4 0.6 0.8 1.0</inputValues>
-          <outputValues>-19.88 -16.52 -12.6 -5.6 -1.4 0.0 2.24 9.52 21.28 28.0 33.6</outputValues>
+          <outputValues>-39.1 -29.32 -19.02 -10.00 -3.14 0.0 3.92 12.55 23.83 37.46 51.5</outputValues>
         </conversion>
       </plugin>
