Commit message: Add LiDAR, ZED spawns in URDF calls, using default topics for now.

File: roboboat/roboboat_description/urdf/actuators.xacro (robot description, xacro)
@@ -9,17 +9,17 @@
     -->
     <!-- Port Bow -->
-    <xacro:thruster_macro robot_namespace="$(arg namespace)" suffix_ns="$(arg suffix_ns)" thruster_id="0">
+    <xacro:thruster_macro robot_namespace="$(arg namespace)" suffix_ns="$(arg suffix_ns)" thruster_id="00">
         <origin xyz="-0.27569 0.32286 -0.29202" rpy="1.570796327 0 2.35619449" />
     </xacro:thruster_macro>
     <!-- Starboard Bow -->
-    <xacro:thruster_macro robot_namespace="$(arg namespace)" suffix_ns="$(arg suffix_ns)" thruster_id="1">
+    <xacro:thruster_macro robot_namespace="$(arg namespace)" suffix_ns="$(arg suffix_ns)" thruster_id="01">
         <origin xyz="0.27569 0.32286 -0.29202" rpy="1.570796327 0 -2.35619449" />
     </xacro:thruster_macro>
     <!-- Port Stern -->
-    <xacro:thruster_macro robot_namespace="$(arg namespace)" suffix_ns="$(arg suffix_ns)" thruster_id="2">
+    <xacro:thruster_macro robot_namespace="$(arg namespace)" suffix_ns="$(arg suffix_ns)" thruster_id="10">
         <origin xyz="-0.28311 -0.31544 -0.29202" rpy="1.570796327 0 -2.35619449" />
     </xacro:thruster_macro>
     <!-- Starboard Stern -->
-    <xacro:thruster_macro robot_namespace="$(arg namespace)" suffix_ns="$(arg suffix_ns)" thruster_id="3">
+    <xacro:thruster_macro robot_namespace="$(arg namespace)" suffix_ns="$(arg suffix_ns)" thruster_id="11">
         <origin xyz="0.28311 -0.31544 -0.29202" rpy="1.570796327 0 2.35619449" />
     </xacro:thruster_macro>

File: roboboat/roboboat_description/urdf/sensors.xacro (robot description, xacro)
@@ -24,49 +24,65 @@
       rpy="$(optenv ROBOBOAT_NAVSAT_UBLOX_RPY 0.0 0.0 0.0)" />
     </joint>
-    <!-- IMU -->
-    <gazebo>
-      <plugin name="imu_controller" filename="libhector_gazebo_ros_imu.so">
-        <robotNamespace>/$(arg namespace)</robotNamespace>
-        <updateRate>50.0</updateRate>
-        <bodyName>$(arg suffix_ns)imu_link</bodyName>
-        <frameId>$(arg suffix_ns)imu_link</frameId>
-        <topicName>/$(arg suffix_ns)imu/data_raw</topicName>
-        <accelDrift>0.005 0.005 0.005</accelDrift>
-        <accelGaussianNoise>0.005 0.005 0.005</accelGaussianNoise>
-        <rateDrift>0.005 0.005 0.005 </rateDrift>
-        <rateGaussianNoise>0.005 0.005 0.005 </rateGaussianNoise>
-        <headingDrift>0.005</headingDrift>
-        <headingGaussianNoise>0.005</headingGaussianNoise>
-      </plugin>
-    </gazebo>
-    <link name="$(arg suffix_ns)imu_link" />
-    <joint name="$(arg suffix_ns)imu_joint" type="fixed">
-      <origin xyz="$(optenv ROBOBOAT_IMU_UM6_XYZ -0.1397 0.0 0)" rpy="$(optenv ROBOBOAT_IMU_UM6_RPY 0 0.0 0.0)" />
-      <parent link="$(arg suffix_ns)base_link" />
-      <child link="$(arg suffix_ns)imu_link" />
-    </joint>
-    <!-- Magnetometer -->
-    <gazebo>
-      <plugin name="mag_controller" filename="libhector_gazebo_ros_magnetic.so">
-        <updateRate>50</updateRate>
-        <robotNamespace>/$(arg namespace)</robotNamespace>
-        <bodyName>$(arg suffix_ns)imu_link</bodyName>
-        <frameId>$(arg suffix_ns)imu_link</frameId>
-        <topicName>/$(arg suffix_ns)imu/mag</topicName>
-        <referenceHeading>90</referenceHeading>
-        <drift>0.0005 0.0005 0.0005</drift>
-        <gaussianNoise>0.025 0.025 0.025</gaussianNoise>
-      </plugin>
-    </gazebo>
-    <!-- Mount a Perfect Pose 3D sensor. -->
-    <gazebo>
-      <plugin filename="libgazebo_ros_p3d.so" name="groundtruth_sim">
-        <updateRate>20.0</updateRate>
-        <robotNamespace>/$(arg namespace)</robotNamespace>
-        <bodyName>$(arg suffix_ns)base_link</bodyName>
-        <topicName>/$(arg suffix_ns)pose_gt</topicName>
-        <gaussianNoise>0.0</gaussianNoise>
-        <frameName>world</frameName>
-      </plugin>
-    </gazebo>
-  </robot>
+  <!-- IMU -->
+  <gazebo>
+    <plugin name="imu_controller" filename="libhector_gazebo_ros_imu.so">
+      <robotNamespace>/$(arg namespace)</robotNamespace>
+      <updateRate>50.0</updateRate>
+      <bodyName>$(arg suffix_ns)imu_link</bodyName>
+      <frameId>$(arg suffix_ns)imu_link</frameId>
+      <topicName>/$(arg suffix_ns)imu/data_raw</topicName>
+      <accelDrift>0.005 0.005 0.005</accelDrift>
+      <accelGaussianNoise>0.005 0.005 0.005</accelGaussianNoise>
+      <rateDrift>0.005 0.005 0.005 </rateDrift>
+      <rateGaussianNoise>0.005 0.005 0.005 </rateGaussianNoise>
+      <headingDrift>0.005</headingDrift>
+      <headingGaussianNoise>0.005</headingGaussianNoise>
+    </plugin>
+  </gazebo>
+  <link name="$(arg suffix_ns)imu_link" />
+  <joint name="$(arg suffix_ns)imu_joint" type="fixed">
+    <origin xyz="$(optenv ROBOBOAT_IMU_UM6_XYZ -0.1397 0.0 0)" rpy="$(optenv ROBOBOAT_IMU_UM6_RPY 0 0.0 0.0)" />
+    <parent link="$(arg suffix_ns)base_link" />
+    <child link="$(arg suffix_ns)imu_link" />
+  </joint>
+  <!-- Magnetometer -->
+  <gazebo>
+    <plugin name="mag_controller" filename="libhector_gazebo_ros_magnetic.so">
+      <updateRate>50</updateRate>
+      <robotNamespace>/$(arg namespace)</robotNamespace>
+      <bodyName>$(arg suffix_ns)imu_link</bodyName>
+      <frameId>$(arg suffix_ns)imu_link</frameId>
+      <topicName>/$(arg suffix_ns)imu/mag</topicName>
+      <referenceHeading>90</referenceHeading>
+      <drift>0.0005 0.0005 0.0005</drift>
+      <gaussianNoise>0.025 0.025 0.025</gaussianNoise>
+    </plugin>
+  </gazebo>
+  <!-- Mount a Perfect Pose 3D sensor. -->
+  <gazebo>
+    <plugin filename="libgazebo_ros_p3d.so" name="groundtruth_sim">
+      <updateRate>20.0</updateRate>
+      <robotNamespace>/$(arg namespace)</robotNamespace>
+      <bodyName>$(arg suffix_ns)base_link</bodyName>
+      <topicName>/$(arg suffix_ns)pose_gt</topicName>
+      <gaussianNoise>0.0</gaussianNoise>
+      <frameName>world</frameName>
+    </plugin>
+  </gazebo>
+  <!-- Bow ZED-->
+  <xacro:vision_macro robot_namespace="$(arg namespace)" suffix_ns="$(arg suffix_ns)" zed_id="0">
+      <origin xyz="0 0.33476 0.16129" rpy="1.5708 0 -3.1416" />
+  </xacro:vision_macro>
+  <!-- Stern ZED-->
+  <xacro:vision_macro robot_namespace="$(arg namespace)" suffix_ns="$(arg suffix_ns)" zed_id="1">
+      <origin xyz="0 -0.33476 0.16129" rpy="1.5708 0 0" />
+  </xacro:vision_macro>
+  <!-- Bow LiDAR-->
+  <xacro:lidar_macro robot_namespace="$(arg namespace)" suffix_ns="$(arg suffix_ns)" lidar_id="0">
+      <origin xyz="0 0.4399 0.07275" rpy="1.5708 0 3.1416" />
+  </xacro:lidar_macro>
+  <!-- Stern LiDAR-->
+  <xacro:lidar_macro robot_namespace="$(arg namespace)" suffix_ns="$(arg suffix_ns)" lidar_id="1">
+      <origin xyz="0 -0.4399 0.07275" rpy="1.5708 0 0" />
+  </xacro:lidar_macro>
+</robot>

File: roboboat/roboboat_description/urdf/snippets.xacro (robot description, xacro)
@@ -101,3 +101,174 @@
     </gazebo>
   </xacro:macro>
+  <!-- MACRO FOR ZED  -->
+  <!--
+    ZED should be initialized in sensors.xacro
+  -->
+  <xacro:macro name="vision_macro" params="robot_namespace suffix_ns zed_id *origin">
+    <!--
+    Dummy link as place holder for the ZED frame.
+    -->
+    <link name="${suffix_ns}zed_${zed_id}">
+      <visual>
+        <geometry>
+          <mesh filename="package://roboboat_description/meshes/base_link_to_zed.STL" />
+        </geometry>
+        <material
+          name="">
+          <color
+            rgba="1 0.949019607843137 0.898039215686275 1" />
+        </material>
+      </visual>
+      <inertial>
+        <origin
+          xyz="0 0 0"
+          rpy="0 0 0" />
+        <mass
+          value="0.60195216377255" />
+        <inertia
+          ixx="9.20940270137913E-05"
+          ixy="-2.6019949675702E-12"
+          ixz="-1.04112177713517E-13"
+          iyy="0.00145803695982764"
+          iyz="-3.92535178970676E-08"
+          izz="0.00144201732186554" />
+      </inertial>
+    </link>
+    <!-- Joint between zed link and vehicle base link -->
+    <joint name="${suffix_ns}zed_${zed_id}_joint" type="continuous">
+      <xacro:insert_block name="origin" />
+      <axis xyz="0 0 1" />
+      <parent link="${suffix_ns}base_link" />
+      <child link="${suffix_ns}zed_${zed_id}" />
+    </joint>
+    <gazebo reference="${suffix_ns}zed_${zed_id}">
+      <sensor type="multicamera" name="stereo_camera">
+        <update_rate>30.0</update_rate>
+        <camera name="left">
+          <horizontal_fov>1.3962634</horizontal_fov>
+          <image>
+            <width>800</width>
+            <height>800</height>
+            <format>R8G8B8</format>
+          </image>
+          <clip>
+            <near>0.02</near>
+            <far>300</far>
+          </clip>
+          <noise>
+            <type>gaussian</type>
+            <mean>0.0</mean>
+            <stddev>0.007</stddev>
+          </noise>
+        </camera>
+        <camera name="right">
+          <pose>0 -0.07 0 0 0 0</pose>
+          <horizontal_fov>1.3962634</horizontal_fov>
+          <image>
+            <width>800</width>
+            <height>800</height>
+            <format>R8G8B8</format>
+          </image>
+          <clip>
+            <near>0.02</near>
+            <far>300</far>
+          </clip>
+          <noise>
+            <type>gaussian</type>
+            <mean>0.0</mean>
+            <stddev>0.007</stddev>
+          </noise>
+        </camera>
+        <plugin name="${suffix_ns}ZED_${zed_id}_controller" filename="libgazebo_ros_multicamera.so">
+          <alwaysOn>true</alwaysOn>
+          <updateRate>0.0</updateRate>
+          <cameraName>multisense_sl/camera</cameraName>
+          <imageTopicName>image_raw</imageTopicName>
+          <cameraInfoTopicName>camera_info</cameraInfoTopicName>
+          <frameName>left_camera_optical_frame</frameName>
+          <!--<rightFrameName>right_camera_optical_frame</rightFrameName>-->
+          <hackBaseline>0.07</hackBaseline>
+          <distortionK1>0.0</distortionK1>
+          <distortionK2>0.0</distortionK2>
+          <distortionK3>0.0</distortionK3>
+          <distortionT1>0.0</distortionT1>
+          <distortionT2>0.0</distortionT2>
+        </plugin>
+      </sensor>
+    </gazebo>
+  </xacro:macro>
+  <xacro:macro name="lidar_macro" params="robot_namespace suffix_ns lidar_id *origin">
+    <!--
+    Dummy link as place holder for the lidar frame.
+    -->
+    <link name="${suffix_ns}lidar_${lidar_id}">
+      <visual>
+        <geometry>
+          <mesh filename="package://roboboat_description/meshes/base_link_to_laser.STL" />
+        </geometry>
+        <material
+        name="">
+        <color
+          rgba="0.1098 0.1098 0.1098 1" />
+        </material>
+      </visual>
+      <inertial>
+        <origin
+          xyz="0 0 0"
+          rpy="0 0 0" />
+        <mass
+          value="0.48577" />
+        <inertia
+          ixx="0.00018166"
+          ixy="-9.1879E-15"
+          ixz="-3.6642E-18"
+          iyy="0.00025601"
+          iyz="3.3496E-07"
+          izz="0.00018167" />
+      </inertial>
+    </link>
+    <!-- Joint between zed link and vehicle base link -->
+    <joint name="${suffix_ns}lidar_${lidar_id}_joint" type="continuous">
+      <xacro:insert_block name="origin" />
+      <axis xyz="0 0 1" />
+      <parent link="${suffix_ns}base_link" />
+      <child link="${suffix_ns}lidar_${lidar_id}" />
+    </joint>
+    <!-- LiDAR -->
+    <gazebo reference="${suffix_ns}lidar_${lidar_id}">
+      <sensor type="ray" name="head_hokuyo_sensor">
+        <pose>0 0 0 0 0 0</pose>
+        <visualize>false</visualize>
+        <update_rate>40</update_rate>
+        <ray>
+          <scan>
+            <horizontal>
+              <samples>720</samples>
+              <resolution>1</resolution>
+              <min_angle>-1.570796</min_angle>
+              <max_angle>1.570796</max_angle>
+            </horizontal>
+          </scan>
+          <range>
+            <min>0.10</min>
+            <max>30.0</max>
+            <resolution>0.01</resolution>
+          </range>
+          <noise>
+            <type>gaussian</type>
+            <!-- Noise parameters based on published spec for Hokuyo laser
+                 achieving "+-30mm" accuracy at range < 10m.  A mean of 0.0m and
+                 stddev of 0.01m will put 99.7% of samples within 0.03m of the true
+                 reading. -->
+            <mean>0.0</mean>
+            <stddev>0.01</stddev>
+          </noise>
+        </ray>
+        <plugin name="gazebo_ros_head_hokuyo_controller" filename="libgazebo_ros_laser.so">
+          <topicName>/rrbot/laser/scan</topicName>
+          <frameName>hokuyo_link</frameName>
+        </plugin>
+      </sensor>
+    </gazebo>
+  </xacro:macro>
 </robot>
