Commit message: Adjusting liar macro, adding PCL service call node to get assembled combined point clouds. Need to populate points.

File: roboboat/roboboat_description/urdf/sensors.xacro (robot description, xacro)
@@ -72,5 +72,5 @@
   <!-- Bow ZED-->
   <xacro:vision_macro robot_namespace="$(arg namespace)" suffix_ns="$(arg suffix_ns)" zed_id="0">
-      <origin xyz="0 0.33476 0.16129" rpy="1.5708 0 -3.1416" />
+      <origin xyz="0 0.33476 0.16129" rpy="1.5708 0 -3.14159" />
   </xacro:vision_macro>
   <!-- Stern ZED-->
@@ -80,5 +80,5 @@
   <!-- Bow LiDAR-->
   <xacro:lidar_macro robot_namespace="$(arg namespace)" suffix_ns="$(arg suffix_ns)" lidar_id="0">
-      <origin xyz="0 0.4399 0.07275" rpy="1.5708 0 3.1416" />
+      <origin xyz="0 0.4399 0.07275" rpy="1.5708 0 3.14159" />
   </xacro:lidar_macro>
   <!-- Stern LiDAR-->

File: roboboat/roboboat_description/urdf/snippets.xacro (robot description, xacro)
@@ -218,10 +218,10 @@
             <alwaysOn>true</alwaysOn>
             <updateRate>1.0</updateRate>
-            <cameraName>bowPoints_ir</cameraName>
+            <cameraName>bowPoints</cameraName>
             <imageTopicName>/bowPoints/color/image_raw</imageTopicName>
             <cameraInfoTopicName>/bowPoints/color/camera_info</cameraInfoTopicName>
             <depthImageTopicName>/bowPoints/depth/image_raw</depthImageTopicName>
             <depthImageInfoTopicName>/bowPoints/depth/camera_info</depthImageInfoTopicName>
-            <pointCloudTopicName>/bowPoints/depth/points</pointCloudTopicName>
+            <pointCloudTopicName>/cloud</pointCloudTopicName>
             <frameName>bowPoints</frameName>
             <pointCloudCutoff>0.5</pointCloudCutoff>
@@ -322,5 +322,5 @@
             <depthImageTopicName>/sternPoints/depth/image_raw</depthImageTopicName>
             <depthImageInfoTopicName>/sternPoints/depth/camera_info</depthImageInfoTopicName>
-            <pointCloudTopicName>/sternPoints/depth/points</pointCloudTopicName>
+            <pointCloudTopicName>/cloud</pointCloudTopicName>
             <frameName>sternPoints</frameName>
             <pointCloudCutoff>0.5</pointCloudCutoff>
@@ -378,40 +378,84 @@
       <child link="${suffix_ns}lidar_${lidar_id}" />
     </joint>
-    <!-- LiDAR -->
-    <gazebo reference="${suffix_ns}lidar_${lidar_id}">
-      <sensor type="ray" name="head_hokuyo_sensor">
-        <pose>0 0 0 0 0 0</pose>
-        <visualize>false</visualize>
-        <update_rate>40</update_rate>
-        <ray>
-          <scan>
-            <horizontal>
-              <samples>720</samples>
-              <resolution>1</resolution>
-              <min_angle>-1.570796</min_angle>
-              <max_angle>1.570796</max_angle>
-            </horizontal>
-          </scan>
-          <range>
-            <min>0.10</min>
-            <max>30.0</max>
-            <resolution>0.01</resolution>
-          </range>
-          <noise>
-            <type>gaussian</type>
-            <!-- Noise parameters based on published spec for Hokuyo laser
-                 achieving "+-30mm" accuracy at range < 10m.  A mean of 0.0m and
-                 stddev of 0.01m will put 99.7% of samples within 0.03m of the true
-                 reading. -->
-            <mean>0.0</mean>
-            <stddev>0.01</stddev>
-          </noise>
-        </ray>
-        <plugin name="gazebo_ros_head_hokuyo_controller" filename="libgazebo_ros_laser.so">
-          <topicName>/laser/scan/${lidar_id}</topicName>
-          <frameName>hokuyo_link</frameName>
-        </plugin>
-      </sensor>
-    </gazebo>
+    <!-- Bow -->
+    <xacro:if value="${lidar_id == 0}">
+      <!-- LiDAR -->
+      <gazebo reference="${suffix_ns}lidar_${lidar_id}">
+        <sensor type="ray" name="head_hokuyo_sensor">
+          <pose>0 0.4399 0.07275 1.5708 0 3.14159</pose>
+          <visualize>false</visualize>
+          <update_rate>40</update_rate>
+          <ray>
+            <scan>
+              <horizontal>
+                <samples>720</samples>
+                <resolution>1</resolution>
+                <min_angle>-1.570796</min_angle>
+                <max_angle>1.570796</max_angle>
+              </horizontal>
+            </scan>
+            <range>
+              <min>0.10</min>
+              <max>30.0</max>
+              <resolution>0.01</resolution>
+            </range>
+            <noise>
+              <type>gaussian</type>
+              <!-- Noise parameters based on published spec for Hokuyo laser
+                   achieving "+-30mm" accuracy at range < 10m.  A mean of 0.0m and
+                   stddev of 0.01m will put 99.7% of samples within 0.03m of the true
+                   reading. -->
+              <mean>0.0</mean>
+              <stddev>0.01</stddev>
+            </noise>
+          </ray>
+          <plugin name="gazebo_ros_head_hokuyo_controller" filename="libgazebo_ros_laser.so">
+            <!-- <topicName>/laser/scan/${lidar_id}</topicName> -->
+            <topicName>/scan</topicName>
+            <frameName>hokuyo_link_${lidar_id}</frameName>
+          </plugin>
+        </sensor>
+      </gazebo>
+    </xacro:if>
+    <!-- Stern -->
+    <xacro:if value="${lidar_id == 1}">
+      <!-- LiDAR -->
+      <gazebo reference="${suffix_ns}lidar_${lidar_id}">
+        <sensor type="ray" name="head_hokuyo_sensor">
+          <pose>0 -0.4399 0.07275 1.5708 0 0</pose>
+          <visualize>false</visualize>
+          <update_rate>40</update_rate>
+          <ray>
+            <scan>
+              <horizontal>
+                <samples>720</samples>
+                <resolution>1</resolution>
+                <min_angle>-1.570796</min_angle>
+                <max_angle>1.570796</max_angle>
+              </horizontal>
+            </scan>
+            <range>
+              <min>0.10</min>
+              <max>30.0</max>
+              <resolution>0.01</resolution>
+            </range>
+            <noise>
+              <type>gaussian</type>
+              <!-- Noise parameters based on published spec for Hokuyo laser
+                   achieving "+-30mm" accuracy at range < 10m.  A mean of 0.0m and
+                   stddev of 0.01m will put 99.7% of samples within 0.03m of the true
+                   reading. -->
+              <mean>0.0</mean>
+              <stddev>0.01</stddev>
+            </noise>
+          </ray>
+          <plugin name="gazebo_ros_head_hokuyo_controller" filename="libgazebo_ros_laser.so">
+            <!-- <topicName>/laser/scan/${lidar_id}</topicName> -->
+            <topicName>/scan</topicName>
+            <frameName>hokuyo_link_${lidar_id}</frameName>
+          </plugin>
+        </sensor>
+      </gazebo>
+    </xacro:if>
   </xacro:macro>
 </robot>
