Commit message: Updates
Updated the Lee Controller gains. Also, updated the flamewheel_f450.yaml and f450.xacro on some parameters.

File: f450_simulator/f450_description/urdf/f450.xacro (robot description, xacro)
@@ -22,23 +22,27 @@
   <xacro:property name="rotor_velocity_slowdown_sim" value="10" />
   <xacro:property name="use_mesh_file" value="true" />
-  <xacro:property name="mesh_file" value="/rotors_description/meshes/base_link.STL" />
-  <xacro:property name="mass" value="1.92" /> <!-- [kg] -->
-  <xacro:property name="body_width" value="0.401" /> <!-- [m] -->
-  <xacro:property name="body_height" value="0.233" /> <!-- [m] -->
-  <xacro:property name="mass_rotor" value="0.009" /> <!-- [kg] -->
-  <xacro:property name="arm_length" value="0.2255" /> <!-- [m] -->
-  <xacro:property name="rotor_offset_top" value="0.01" /> <!-- [m] -->
+  <xacro:property name="mesh_file" value="package://rotors_description/meshes/base_link.STL" />
+  <xacro:property name="mass" value="1.43508388852705" /> <!-- [kg] -->
+  <xacro:property name="body_width" value="0.36" /> <!-- [m] -->
+  <xacro:property name="body_height" value="0.218" /> <!-- [m] -->
+  <xacro:property name="mass_rotor" value="0.0124" /> <!-- [kg] -->
+  <xacro:property name="arm_length" value="0.185" /> <!-- [m] -->
+  <xacro:property name="rotor_offset_top" value="0.045" /> <!-- [m] -->
   <xacro:property name="radius_rotor" value="0.127" /> <!-- [m] -->
-  <xacro:property name="motor_constant" value="8.54858e-06" /> <!-- [kg m/s^2] -->
-  <xacro:property name="moment_constant" value="0.016" /> <!-- [m] -->
+  <xacro:property name="motor_constant" value="8.54858e-06" /> <!-- [kg m/s^2] Have not changed -->
+  <xacro:property name="moment_constant" value="0.016" /> <!-- [m] Have not changed -->
   <xacro:property name="time_constant_up" value="0.0125" /> <!-- [s] -->
   <xacro:property name="time_constant_down" value="0.025" /> <!-- [s] -->
-  <xacro:property name="max_rot_velocity" value="838" /> <!-- [rad/s] -->
+  <xacro:property name="max_rot_velocity" value="838" /> <!-- [rad/s] Have not changed -->
   <xacro:property name="rotor_drag_coefficient" value="8.06428e-05" />
   <xacro:property name="rolling_moment_coefficient" value="0.000001" />
   <!-- Property Blocks -->
   <xacro:property name="body_inertia">
-    <inertia ixx="0.002" ixy="0.0" ixz="0.0" iyy="0.003" iyz="0.0" izz="0.002" /> <!-- [kg m^2] [kg m^2] [kg m^2] [kg m^2] [kg m^2] [kg m^2] -->
+    <inertia ixx="0.003" ixy="0.0" ixz="0.0" iyy="0.0015" iyz="0.0" izz="0.004" /> <!-- [kg m^2] [kg m^2] [kg m^2] [kg m^2] [kg m^2] [kg m^2] -->
   </xacro:property>
+  <!--
+  <xacro:property name="body_inertia">
+    <inertia ixx="0.003034335338584" ixy="0.000000045751812000923" ixz="0.000000158361637575774" iyy="0.001496545528055" iyz="-0.000000483515340559471" izz="0.00381045049143025" />
+  -->
   <!-- inertia of a single rotor, assuming it is a cuboid. Height=3mm, width=15mm -->
   <xacro:property name="rotor_inertia">
@@ -58,5 +62,5 @@
   </xacro:multirotor_base_macro>
   <!-- Instantiate rotors -->
-    <xacro:vertical_rotor
+  <xacro:vertical_rotor
     robot_namespace="${namespace}"
     suffix="front"
@@ -73,5 +77,5 @@
     rotor_drag_coefficient="${rotor_drag_coefficient}"
     rolling_moment_coefficient="${rolling_moment_coefficient}"
-    color="Black"
+    color="Red"
     use_own_mesh="false"
     mesh="">
@@ -94,8 +98,8 @@
     rotor_drag_coefficient="${rotor_drag_coefficient}"
     rolling_moment_coefficient="${rolling_moment_coefficient}"
-    color="Black"
+    color="Blue"
     use_own_mesh="false"
     mesh="">
-    <origin xyz="0.1581 0.0355 ${rotor_offset_top}" rpy="0 0 0" />
+    <origin xyz="0 ${arm_length} ${rotor_offset_top}" rpy="0 0 0" />
     <xacro:insert_block name="rotor_inertia" />
   </xacro:vertical_rotor>
@@ -115,5 +119,5 @@
     rotor_drag_coefficient="${rotor_drag_coefficient}"
     rolling_moment_coefficient="${rolling_moment_coefficient}"
-    color="Black"
+    color="Blue"
     use_own_mesh="false"
     mesh="">
@@ -136,5 +140,5 @@
     rotor_drag_coefficient="${rotor_drag_coefficient}"
     rolling_moment_coefficient="${rolling_moment_coefficient}"
-    color="Black"
+    color="Blue"
     use_own_mesh="false"
     mesh="">
@@ -142,13 +146,3 @@
     <xacro:insert_block name="rotor_inertia" />
   </xacro:vertical_rotor>
-  <!-- Inputting Cameras and Lidar -->
-  <!-- Mount a VI-sensor in front of the Firefly. -->
-  <xacro:vi_sensor_macro
-    namespace="${namespace}/vi_sensor"
-    parent_link="${namespace}/base_link"
-    enable_cameras="true"
-    enable_depth="true"
-    enable_ground_truth="true">
-    <origin xyz="0.000865 0.01907 0.0821" rpy="0.0 0.1 0.0" />
-  </xacro:vi_sensor_macro>
 </robot>

Commit message: Updates to f450_description fixed package

File: f450_simulator/f450_description/urdf/f450.xacro (robot description, xacro)
@@ -22,5 +22,5 @@
   <xacro:property name="rotor_velocity_slowdown_sim" value="10" />
   <xacro:property name="use_mesh_file" value="true" />
-  <xacro:property name="mesh_file" value="package://rotors_description/meshes/base_link.STL" />
+  <xacro:property name="mesh_file" value="package://f450_description/meshes/base_link.STL" />
   <xacro:property name="mass" value="1.43508388852705" /> <!-- [kg] -->
   <xacro:property name="body_width" value="0.36" /> <!-- [m] -->
@@ -50,5 +50,5 @@
   </xacro:property>
   <!-- Included URDF Files -->
-  <xacro:include filename="$(find rotors_description)/urdf/multirotor_base.xacro" />
+  <xacro:include filename="$(find f450_description)/urdf/multirotor_base.xacro" />
   <!-- Instantiate multirotor_base_macro once -->
   <xacro:multirotor_base_macro

File: f450_simulator/f450_description/urdf/f450_base.xacro (robot description, xacro)
@@ -16,8 +16,8 @@
   limitations under the License.
 -->
-<robot name="f450" xmlns:xacro="http://ros.org/wiki/xacro">
-  <xacro:include filename="$(find rotors_description)/urdf/component_snippets.xacro" />
+<robot name="f450_base" xmlns:xacro="http://ros.org/wiki/xacro">
+  <xacro:include filename="$(find f450_description)/urdf/component_snippets.xacro" />
   <!-- Instantiate FlameWheel_F450 "mechanics" -->
-  <xacro:include filename="$(find rotors_description)/urdf/f450.xacro" />
+  <xacro:include filename="$(find f450_description)/urdf/f450.xacro" />
   <!-- Instantiate a controller. -->
   <xacro:controller_plugin_macro namespace="${namespace}" imu_sub_topic="imu" />

Commit message: Updates to propeller locations and updates to the lee_controller_f450.yaml as well some other minor updates
Unfortunately Brennan and I are having trouble with making the transition from rotors_... to f450_... . We know this is something we can figure out, but it just is taking more time than we were hoping for. Also, for the lee_controller_f450.yaml, I am seeing more results with how I have tried this new approach that Dr. Vaughan sent over to me today. It appears that I am seeing more of the trend that is letting me control the drone much better

File: f450_simulator/f450_description/urdf/f450.xacro (robot description, xacro)
@@ -22,11 +22,11 @@
   <xacro:property name="rotor_velocity_slowdown_sim" value="10" />
   <xacro:property name="use_mesh_file" value="true" />
-  <xacro:property name="mesh_file" value="package://f450_description/meshes/base_link.STL" />
+  <xacro:property name="mesh_file" value="package://rotors_description/meshes/base_link.STL" />
   <xacro:property name="mass" value="1.43508388852705" /> <!-- [kg] -->
-  <xacro:property name="body_width" value="0.36" /> <!-- [m] -->
+  <xacro:property name="body_width" value="0.4" /> <!-- [m] -->
   <xacro:property name="body_height" value="0.218" /> <!-- [m] -->
   <xacro:property name="mass_rotor" value="0.0124" /> <!-- [kg] -->
-  <xacro:property name="arm_length" value="0.185" /> <!-- [m] -->
-  <xacro:property name="rotor_offset_top" value="0.045" /> <!-- [m] -->
+  <xacro:property name="arm_length" value="0.159" /> <!-- [m] -->
+  <xacro:property name="rotor_offset_top" value="0.065" /> <!-- [m] -->
   <xacro:property name="radius_rotor" value="0.127" /> <!-- [m] -->
   <xacro:property name="motor_constant" value="8.54858e-06" /> <!-- [kg m/s^2] Have not changed -->
@@ -50,5 +50,5 @@
   </xacro:property>
   <!-- Included URDF Files -->
-  <xacro:include filename="$(find f450_description)/urdf/multirotor_base.xacro" />
+  <xacro:include filename="$(find rotors_description)/urdf/multirotor_base.xacro" />
   <!-- Instantiate multirotor_base_macro once -->
   <xacro:multirotor_base_macro
@@ -80,5 +80,5 @@
     use_own_mesh="false"
     mesh="">
-    <origin xyz="${arm_length} 0 ${rotor_offset_top}" rpy="0 0 0" />
+    <origin xyz="${arm_length} ${arm_length} ${rotor_offset_top}" rpy="0 0 0" />
     <xacro:insert_block name="rotor_inertia" />
   </xacro:vertical_rotor>
@@ -98,8 +98,8 @@
     rotor_drag_coefficient="${rotor_drag_coefficient}"
     rolling_moment_coefficient="${rolling_moment_coefficient}"
-    color="Blue"
+    color="Black"
     use_own_mesh="false"
     mesh="">
-    <origin xyz="0 ${arm_length} ${rotor_offset_top}" rpy="0 0 0" />
+    <origin xyz="-${arm_length} ${arm_length} ${rotor_offset_top}" rpy="0 0 0" />
     <xacro:insert_block name="rotor_inertia" />
   </xacro:vertical_rotor>
@@ -119,8 +119,8 @@
     rotor_drag_coefficient="${rotor_drag_coefficient}"
     rolling_moment_coefficient="${rolling_moment_coefficient}"
-    color="Blue"
+    color="Red"
     use_own_mesh="false"
     mesh="">
-    <origin xyz="-${arm_length} 0 ${rotor_offset_top}" rpy="0 0 0" />
+    <origin xyz="-${arm_length} -${arm_length} ${rotor_offset_top}" rpy="0 0 0" />
     <xacro:insert_block name="rotor_inertia" />
   </xacro:vertical_rotor>
@@ -140,8 +140,8 @@
     rotor_drag_coefficient="${rotor_drag_coefficient}"
     rolling_moment_coefficient="${rolling_moment_coefficient}"
-    color="Blue"
+    color="Black"
     use_own_mesh="false"
     mesh="">
-    <origin xyz="0 -${arm_length} ${rotor_offset_top}" rpy="0 0 0" />
+    <origin xyz="${arm_length} -${arm_length} ${rotor_offset_top}" rpy="0 0 0" />
     <xacro:insert_block name="rotor_inertia" />
   </xacro:vertical_rotor>

File: f450_simulator/f450_description/urdf/f450_base.xacro (robot description, xacro)
@@ -16,8 +16,8 @@
   limitations under the License.
 -->
-<robot name="f450_base" xmlns:xacro="http://ros.org/wiki/xacro">
-  <xacro:include filename="$(find f450_description)/urdf/component_snippets.xacro" />
+<robot name="f450" xmlns:xacro="http://ros.org/wiki/xacro">
+  <xacro:include filename="$(find rotors_description)/urdf/component_snippets.xacro" />
   <!-- Instantiate FlameWheel_F450 "mechanics" -->
-  <xacro:include filename="$(find f450_description)/urdf/f450.xacro" />
+  <xacro:include filename="$(find rotors_description)/urdf/f450.xacro" />
   <!-- Instantiate a controller. -->
   <xacro:controller_plugin_macro namespace="${namespace}" imu_sub_topic="imu" />

Commit message: Update to f450.xacro mass

File: f450_simulator/f450_description/urdf/f450.xacro (robot description, xacro)
@@ -23,5 +23,5 @@
   <xacro:property name="use_mesh_file" value="true" />
   <xacro:property name="mesh_file" value="package://rotors_description/meshes/base_link.STL" />
-  <xacro:property name="mass" value="1.43508388852705" /> <!-- [kg] -->
+  <xacro:property name="mass" value="1.92" /> <!-- [kg] -->
   <xacro:property name="body_width" value="0.4" /> <!-- [m] -->
   <xacro:property name="body_height" value="0.218" /> <!-- [m] -->
