Commit message: RotorS_Sim: f450 drone updates for all the sensors in correct locations and all transforms work correctly
Drone is now ready to go through any simulation that it would need to go through

File: rotors_simulator/rotors_description/urdf/component_snippets.xacro (robot description, xacro)
@@ -54,7 +54,7 @@
       </xacro:if>
       <inertial>
-        <mass value="1e-5" />
-        <origin xyz="0 0 0" rpy="0 0 0" />
-        <inertia ixx="1e-6" ixy="0" ixz="0" iyy="1e-6" iyz="0" izz="1e-6" />
+        <mass value="1e-1000" />
+        <origin xyz="0 0 0" rpy="0 0 0" />
+        <inertia ixx="1e-20" ixy="0" ixz="0" iyy="1e-6" iyz="0" izz="1e-6" />
       </inertial>
     </link>
@@ -551,7 +551,7 @@
     </gazebo>
   </xacro:macro>
-  <!-- VI sensor macros -->
-  <!-- Macro to add a VI-sensor camera. -->
-  <xacro:macro name="vi_sensor_camera_macro"
+  <!-- oak_d sensor macros -->
+  <!-- Macro to add a oak_d-sensor camera. -->
+  <xacro:macro name="oak_d_sensor_camera_macro"
     params="namespace parent_link camera_suffix frame_rate *origin">
     <xacro:camera_macro
@@ -569,14 +569,14 @@
       noise_stddev="0.007"
       enable_visual="true">
-      <mesh filename="package://rotors_description/meshes/vi_camera.dae" scale="1 1 1" />
+      <mesh filename="package://rotors_description/meshes/oak_d.STL" scale=".1 .1 .1" />
       <xacro:insert_block name="origin" />
     </xacro:camera_macro>
   </xacro:macro>
-  <!-- Macro to add a VI-sensor stereo camera. -->
-  <xacro:macro name="vi_sensor_stereo_camera_macro"
+  <!-- Macro to add a oak_d-sensor stereo camera. -->
+  <xacro:macro name="oak_d_sensor_stereo_camera_macro"
     params="namespace parent_link frame_rate origin_offset_x baseline_y origin_offset_z max_range">
     <xacro:stereo_camera_macro
       namespace="${namespace}"
-      camera_name="vi_sensor"
+      camera_name="oak_d_sensor"
       parent_link="${parent_link}"
       frame_rate="${frame_rate}"
@@ -596,6 +596,6 @@
     </xacro:stereo_camera_macro>
   </xacro:macro>
-  <!-- Macro to add a depth camera on the VI-sensor. -->
-  <xacro:macro name="vi_sensor_depth_macro"
+  <!-- Macro to add a depth camera on the oak_d-sensor. -->
+  <xacro:macro name="oak_d_sensor_depth_macro"
     params="namespace parent_link camera_suffix frame_rate max_range *origin">
     <link name="${namespace}/camera_${camera_suffix}_link">
@@ -665,18 +665,18 @@
     </gazebo>
   </xacro:macro>
-  <!-- VI-Sensor Macro -->
-  <xacro:macro name="vi_sensor_macro" params="namespace parent_link enable_cameras enable_depth enable_ground_truth *origin">
-    <!-- Vi Sensor Link -->
-    <link name="${namespace}/vi_sensor_link">
+  <!-- oak_d-Sensor Macro -->
+  <xacro:macro name="oak_d_sensor_macro" params="namespace parent_link enable_cameras enable_depth enable_ground_truth *origin">
+    <!-- oak_d Sensor Link -->
+    <link name="${namespace}/oak_d_sensor_link">
       <collision>
-        <origin xyz="0 0 0" rpy="0 0 0" />
+        <origin xyz="-0.01 -0.055 -0.04" rpy="1.570796327 0 1.570796327" />
         <geometry>
-          <box size="0.03 0.133 0.057" />
+          <mesh filename="package://rotors_description/meshes/oak_d.STL" scale=".001 .001 .001" />
         </geometry>
       </collision>
       <visual>
-        <origin xyz="0 0 0" rpy="0 0 0" />
+        <origin xyz="-0.01 -0.055 -0.04" rpy="1.570796327 0 1.570796327" />
         <geometry>
-          <mesh filename="package://rotors_description/meshes/vi_sensor.dae" scale="1 1 1" />
+          <mesh filename="package://rotors_description/meshes/oak_d.STL" scale=".001 .001 .001" />
         </geometry>
       </visual>
@@ -687,25 +687,25 @@
       </inertial>
     </link>
-    <joint name="${namespace}_vi_sensor_joint" type="fixed">
+    <joint name="${namespace}_oak_d_sensor_joint" type="fixed">
       <xacro:insert_block name="origin" />
       <parent link="${parent_link}" />
-      <child link="${namespace}/vi_sensor_link" />
+      <child link="${namespace}/oak_d_sensor_link" />
     </joint>
     <!-- Cameras -->
     <xacro:if value="${enable_cameras}">
       <!-- Insert stereo pair. -->
-      <xacro:vi_sensor_stereo_camera_macro
-        namespace="${namespace}" parent_link="${namespace}/vi_sensor_link"
-        frame_rate="30.0" origin_offset_x="0.015" baseline_y="${0.055*2}"
+      <xacro:oak_d_sensor_stereo_camera_macro
+        namespace="${namespace}" parent_link="${namespace}/oak_d_sensor_link"
+        frame_rate="30.0" origin_offset_x="0.01" baseline_y="${0.055*1.67}"
         origin_offset_z="0.0065" max_range="30.0">
-      </xacro:vi_sensor_stereo_camera_macro>
+      </xacro:oak_d_sensor_stereo_camera_macro>
     </xacro:if>
     <!-- Depth Sensor -->
     <xacro:if value="${enable_depth}">
-      <xacro:vi_sensor_depth_macro
-        namespace="${namespace}" parent_link="${namespace}/vi_sensor_link"
+      <xacro:oak_d_sensor_depth_macro
+        namespace="${namespace}" parent_link="${namespace}/oak_d_sensor_link"
         camera_suffix="depth" frame_rate="30.0" max_range="30.0">
-        <origin xyz="0.015 0.055 0.0065" rpy="0 0 0" />
-      </xacro:vi_sensor_depth_macro>
+        <origin xyz="0.015 -0 0.0065" rpy="0 0 0" />
+      </xacro:oak_d_sensor_depth_macro>
     </xacro:if>
     <!-- Groundtruth -->
@@ -715,5 +715,5 @@
         namespace="${namespace}/ground_truth"
         odometry_sensor_suffix=""
-        parent_link="${namespace}/vi_sensor_link"
+        parent_link="${namespace}/oak_d_sensor_link"
         pose_topic="pose"
         pose_with_covariance_topic="pose_with_covariance"
@@ -746,5 +746,5 @@
       namespace="${namespace}"
       imu_suffix=""
-      parent_link="${namespace}/vi_sensor_link"
+      parent_link="${namespace}/oak_d_sensor_link"
       imu_topic="imu"
       mass_imu_sensor="0.015"
@@ -899,8 +899,8 @@
 <!-- OUR SENSORS -->
 <!-- Macro to add a LiDAR. -->
-<!-- Macro to add a rpi camera. -->
+<!-- Macro to add the rpi camera. -->
   <!-- Macro to add a camera. -->
-  <xacro:macro name="vi1_sensor_camera_macro"
-    params="namespace parent_link frame_rate origin_offset_x baseline_y origin_offset_z max_range">
+  <xacro:macro name="rpi_sensor_camera_macro"
+    params="namespace parent_link frame_rate *origin max_range">
     <xacro:camera_macro
       namespace="${namespace}"
@@ -908,5 +908,5 @@
       camera_suffix="rpi"
       frame_rate="30"
-      horizontal_fov="1.3962634"
+      horizontal_fov="1.085595"
       image_width="1080"
       image_height="720"
@@ -921,105 +921,13 @@
     </xacro:camera_macro>
   </xacro:macro>
-  <!-- Macro to add a VI-sensor stereo camera. -->
-  <xacro:macro name="vi1_sensor_stereo_camera_macro"
-    params="namespace parent_link frame_rate origin_offset_x baseline_y origin_offset_z max_range">
-    <xacro:stereo_camera_macro
-      namespace="${namespace}"
-      camera_name="vi1_sensor"
-      parent_link="${parent_link}"
-      frame_rate="${frame_rate}"
-      horizontal_fov="1.3962634"
-      image_width="1080"
-      image_height="720"
-      image_format="R8G8B8"
-      min_distance="0.08"
-      max_distance="30"
-      noise_mean="0.0"
-      noise_stddev="0.007"
-      enable_visual="false"
-      origin_offset_x="${origin_offset_x}"
-      baseline_y="${baseline_y}"
-      origin_offset_z="${origin_offset_z}" >
-      <cylinder length="0.01" radius="0.007" />
-    </xacro:stereo_camera_macro>
-  </xacro:macro>
-  <!-- Macro to add a depth camera on the VI1-sensor. -->
-  <xacro:macro name="vi1_sensor_depth_macro"
-    params="namespace parent_link camera_suffix frame_rate max_range *origin">
-    <link name="${namespace}/camera_${camera_suffix}_link">
-      <collision>
-        <origin xyz="0 0 0" rpy="0 0 0" />
-        <geometry>
-          <cylinder length="0.01" radius="0.007" />
-        </geometry>
-      </collision>
-      <inertial>
-        <mass value="1e-1000" />
-        <origin xyz="0 0 0" rpy="0 0 0" />
-        <inertia ixx="1e-6" ixy="0" ixz="0" iyy="1e-6" iyz="0" izz="1e-6" />
-      </inertial>
-    </link>
-    <joint name="${namespace}/camera_${camera_suffix}_joint" type="fixed">
-      <xacro:insert_block name="origin" />
-      <parent link="${parent_link}" />
-      <child link="${namespace}/camera_${camera_suffix}_link" />
-      <limit upper="0" lower="0" effort="0" velocity="0" />
-    </joint>
-    <!-- Optical center of camera -->
-    <link name="${namespace}/camera_${camera_suffix}_optical_center_link" />
-    <joint name="${namespace}/camera_${camera_suffix}_optical_center_joint" type="fixed">
-      <origin xyz="0 0 0" rpy="${-pi/2} 0 ${-pi/2}" />
-      <parent link="${namespace}/camera_${camera_suffix}_link" />
-      <child link="${namespace}/camera_${camera_suffix}_optical_center_link" />
-      <limit upper="0" lower="0" effort="0" velocity="0" />
-    </joint>
-    <gazebo reference="${namespace}/camera_${camera_suffix}_link">
-      <sensor type="depth" name="${namespace}_camera_{camera_suffix}">
-        <always_on>true</always_on>
-        <update_rate>30</update_rate>
-        <camera>
-          <horizontal_fov>2</horizontal_fov>
-          <image>
-            <format>R8G8B8</format>
-            <width>1080</width>
-            <height>720</height>
-          </image>
-          <clip>
-            <near>0.08</near>
-            <far>30</far>
-          </clip>
-        </camera>
-        <plugin name="${namespace}_camera_{camera_suffix}" filename="libgazebo_ros_openni_kinect.so">
-          <robotNamespace>${namespace}</robotNamespace>
-          <alwaysOn>true</alwaysOn>
-          <baseline>0.11</baseline>
-          <updateRate>30</updateRate>
-          <cameraName>camera_${camera_suffix}</cameraName>
-          <imageTopicName>camera/image_raw</imageTopicName>
-          <cameraInfoTopicName>camera/camera_info</cameraInfoTopicName>
-          <depthImageTopicName>depth/disparity</depthImageTopicName>
-          <depthImageCameraInfoTopicName>depth/camera_info</depthImageCameraInfoTopicName>
-          <pointCloudTopicName>depth/points</pointCloudTopicName>
-          <frameName>camera_${camera_suffix}_optical_center_link</frameName>
-          <pointCloudCutoff>0.5</pointCloudCutoff>
-          <pointCloudCutoffMax>30</pointCloudCutoffMax>
-          <distortionK1>0.0</distortionK1>
-          <distortionK2>0.0</distortionK2>
-          <distortionK3>0.0</distortionK3>
-          <distortionT1>0.0</distortionT1>
-          <distortionT2>0.0</distortionT2>
-        </plugin>
-      </sensor>
-    </gazebo>
-  </xacro:macro>
-  <!-- VI1-Sensor Macro -->
-  <xacro:macro name="vi1_sensor_macro" params="namespace parent_link enable_cameras *origin">
-    <!-- Vi1 Sensor Link -->
+  <!-- rpi-Sensor Macro -->
+  <xacro:macro name="rpi_sensor_macro" params="namespace parent_link enable_cameras *origin">
+    <!-- rpi Sensor Link -->
     <link name="${namespace}/rpi_sensor_link">
       <collision>
         <origin xyz="0 0 0" rpy="0 1.570796327 0" />
         <geometry>
-          <box size="0.03 0.03 0.057" />
-        </geometry>
+          <mesh filename="package://rotors_description/meshes/link_7.STL" scale="1 1 1" />
+        </geometry>>
       </collision>
       <visual>
@@ -1035,5 +943,5 @@
       </inertial>
     </link>
-    <joint name="${namespace}_vi1_sensor_joint" type="fixed">
+    <joint name="${namespace}_rpi_sensor_joint" type="fixed">
       <xacro:insert_block name="origin" />
       <parent link="${parent_link}" />
@@ -1043,9 +951,9 @@
     <xacro:if value="${enable_cameras}">
       <!-- Insert Camera. -->
-      <xacro:vi1_sensor_camera_macro
+      <xacro:rpi_sensor_camera_macro
         namespace="${namespace}" parent_link="${namespace}/rpi_sensor_link"
-        frame_rate="30.0" origin_offset_x="0.0" baseline_y="0.0"
-        origin_offset_z="0.0065" max_range="30.0">
-      </xacro:vi1_sensor_camera_macro>
+        frame_rate="30.0" max_range="30.0">
+        <origin xyz="0 0 0" rpy="0 0 0" />
+      </xacro:rpi_sensor_camera_macro>
     </xacro:if>
   </xacro:macro>

File: rotors_simulator/rotors_description/urdf/f450.xacro (robot description, xacro)
@@ -148,6 +148,6 @@
 <!-- Creating Our Own Sensors -->
   <!-- Mount a VI-sensor (OAK-D) in front of the F450 -->
-  <xacro:vi_sensor_macro
-    namespace="${namespace}/vi_sensor"
+  <xacro:oak_d_sensor_macro
+    namespace="${namespace}/oak_d_sensor"
     parent_link="${namespace}/base_link"
     enable_cameras="true"
@@ -155,13 +155,66 @@
     enable_ground_truth="true">
     <origin xyz="0.0 0.08 0.16" rpy="0.0 0.34906585 1.570796327" />
-  </xacro:vi_sensor_macro>
-  <!-- Mount a LiDAR on the Side of the F450 -->
+  </xacro:oak_d_sensor_macro>
+  <!-- Mount LiDAR in front of the F450 -->
+  <joint name="lidar_lite_v3hp_joint" type="fixed">
+    <axis xyz="0 1 0" />
+    <origin xyz="-0.04 0.02 0.071" rpy="1.570796327 1.570796327 0"/>
+    <parent link="${namespace}/base_link"/>
+    <child link="lidar_lite_v3hp"/>
+  </joint>
+  <!-- LiDAR Lite V3HP Laser -->
+  <link name="lidar_lite_v3hp">
+    <collision>
+      <origin xyz="-0.04 0.02 0.02" rpy="0 0 4.71238898"/>
+      <geometry>
+        <mesh filename="package://rotors_description/meshes/link_5.STL"/>
+      </geometry>
+    </collision>
+    <visual>
+      <origin xyz="-0.04 0.02 0.02" rpy="0 0 4.71238898"/>
+      <geometry>
+        <mesh filename="package://rotors_description/meshes/link_5.STL"/>
+      </geometry>
+    </visual>
+    <inertial>
+      <mass value="1e-20" />
+      <origin xyz="0 0 0" rpy="0 0 0"/>
+      <inertia ixx="1e-6" ixy="0" ixz="0" iyy="1e-6" iyz="0" izz="1e-6" />
+    </inertial>
+  </link>
+  <!-- Might be an alternate option
+  <xacro:include filename="lidar.xacro"/>
+  <joint name="lidarGlue" type="fixed">
+    <parent link="${namespace}/base_link"/>
+    <child link="laz_base"/>
+    <origin xyz="0 0 0.1" rpy="0 0 0" />
+  </joint>
+  -->
   <!-- Mount a Raspberry Pi Camera on the Bottom of the F450 -->
-  <xacro:vi1_sensor_macro
-    namespace="${namespace}/vi1_sensor"
+  <xacro:rpi_sensor_macro
+    namespace="${namespace}/rpi_sensor"
     parent_link="${namespace}/base_link"
-    enable_cameras="true"
-    >
-    <origin xyz="0.0 0.0 0.0" rpy="0.0 0.0 0.0" />
-  </xacro:vi1_sensor_macro>
+    enable_cameras="true">
+    <origin xyz="0.0 0.0 0.083" rpy="1.570796327 1.570796327 1.570796327" />
+  </xacro:rpi_sensor_macro>
+  <!-- Other Camera -->
+  <!--
+  <xacro:camera_macro
+    namespace="${namespace}"
+    parent_link="${namespace}/base_link"
+    camera_suffix="left"
+    frame_rate="30"
+    horizontal_fov="2"
+    image_width="1080"
+    image_height="720"
+    image_format="R8G8B8"
+    min_distance="1"
+    max_distance="50"
+    noise_mean="0.0"
+    noise_stddev="0.007"
+    enable_visual="true">
+    <box size="0.02 0.05 0.05" />
+    <origin xyz="${arm_length/3} 0 0" rpy="0 0 0" />
+  </xacro:camera_macro>
+  -->
 </robot>

File: rotors_simulator/rotors_description/urdf/multirotor_base.xacro (robot description, xacro)
@@ -58,7 +58,7 @@
       </visual>
       <collision>
-        <origin xyz="0 0 0.1" rpy="0 0 3.14" />
+        <origin xyz="0 0 0.12" rpy="0 0 3.14" />
         <geometry>
-          <box size="${body_width} ${body_width} ${body_height}" /> <!-- [m] [m] [m] -->
+            <mesh filename="${mesh_file}" scale="1 1 1" />
         </geometry>
       </collision>
